File: KiCad/Exchange_ProofOfConcept/ESP-Unit/ESP-Unit.kicad_sch (KiCad schematic)
At the start: 2 parts, among them U1 ESP32-DEVKITC

Commit message: Changes to be committed: 	new file:   KiCad/Exchange_ProofOfConcept/ESP-Unit/ESP-Unit-backups/ESP-Unit-2024-11-30_004013.zip 	new file:   KiCad/Exchange_ProofOfConcept/ESP-Unit/ESP-Unit-backups/ESP-Unit-2024-11-30_005151.zip 	new file:   KiCad/Exchange_ProofOfConcept/ESP-Unit/ESP-Unit-backups/ESP-Unit-2024-11-30_173159.zip 	new file:   KiCad/Exchange_ProofOfConcept/ESP-Unit/ESP-Unit-backups/ESP-Unit-2024-12-02_225320.zip 	new file:   KiCad/Exchange_ProofOfConcept/ESP-Unit/ESP-Unit-backups/ESP-Unit-2024-12-02_230401.zip 	new file:   KiCad/Exchange_ProofOfConcept/ESP-Unit/ESP-Unit-backups/ESP-Unit-2024-12-02_231401.zip 	new file:   KiCad/Exchange_ProofOfConcept/ESP-Unit/ESP-Unit-backups/ESP-Unit-2024-12-02_232414.zip 	new file:   KiCad/Exchange_ProofOfConcept/ESP-Unit/ESP-Unit-backups/ESP-Unit-2024-12-02_233354.zip 	new file:   KiCad/Exchange_ProofOfConcept/ESP-Unit/ESP-Unit-backups/ESP-Unit-2024-12-04_223019.zip 	new file:   KiCad/Exchange_ProofOfConcept/ESP-Unit/ESP-Unit-backups/ESP-Unit-2024-12-04_223655.zip 	new file:   KiCad/Exchange_ProofOfConcept/ESP-Unit/ESP-Unit-backups/ESP-Unit-2024-12-04_225021.zip 	new file:   KiCad/Exchange_ProofOfConcept/ESP-Unit/ESP-Unit-backups/ESP-Unit-2024-12-04_230524.zip 	new file:   KiCad/Exchange_ProofOfConcept/ESP-Unit/ESP-Unit-backups/ESP-Unit-2024-12-04_231506.zip 	new file:   KiCad/Exchange_ProofOfConcept/ESP-Unit/ESP-Unit-backups/ESP-Unit-2024-12-05_032122.zip 	new file:   KiCad/Exchange_ProofOfConcept/ESP-Unit/ESP-Unit-backups/ESP-Unit-2024-12-06_183750.zip 	new file:   KiCad/Exchange_ProofOfConcept/ESP-Unit/ESP-Unit-backups/ESP-Unit-2024-12-07_112304.zip 	new file:   KiCad/Exchange_ProofOfConcept/ESP-Unit/ESP-Unit-backups/ESP-Unit-2024-12-07_125326.zip 	modified:   KiCad/Exchange_ProofOfConcept/ESP-Unit/ESP-Unit.kicad_pcb 	modified:   KiCad/Exchange_ProofOfConcept/ESP-Unit/ESP-Unit.kicad_prl 	modified:   KiCad/Exchange_ProofOfConcept/ESP-Unit/ESP-Unit.kicad_pro 	modified:   KiCad/Exchange_ProofOfConcept/ESP-Unit/ESP-Unit.k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
Parts:
- removed U1: ESP32-DEVKITC, ESP32-DEVKITC:MODULE_ESP32-DEVKITC, symbol JW_library_sym:ESP32-DEVKITC
- added C1, C4, C5, C6, C8, C9: 0,1uF, Capacitor_THT:C_Disc_D5.0mm_W2.5mm_P2.50mm, symbol Device:C
- added C10, C3: 2n2, Capacitor_THT:C_Disc_D5.0mm_W2.5mm_P2.50mm, symbol Device:C
- added C2: 10uF, Capacitor_THT:C_Disc_D5.0mm_W2.5mm_P2.50mm, symbol Device:C
- added C7: 47uF, Capacitor_THT:CP_Radial_D4.0mm_P2.00mm, symbol Device:C_Polarized_US
- added D1: LED, LED_THT:LED_D5.0mm, symbol Device:LED
- added D2, D3, D4, D5: LED, LED_THT:LED_D3.0mm, symbol Device:LED
- added H1, H2, H3, H4: MountingHole_Pad, MountingHole:MountingHole_3.2mm_M3_Pad_Via, symbol Mechanical:MountingHole_Pad
- added IC1: MT8870DE, Package_DIP:DIP-18_W7.62mm_LongPads, symbol JW_library_sym:MT8870
- added J2: Conn_02x05_Top_Bottom, Connector_PinHeader_2.54mm:PinHeader_2x05_P2.54mm_Vertical, symbol Connector_Generic:Conn_02x05_Top_Bottom
- added J3: Conn_01x07, Connector_PinSocket_2.54mm:PinSocket_1x07_P2.54mm_Vertical, symbol Connector_Generic:Conn_01x07
- added R1: 240, Resistor_THT:R_Axial_DIN0207_L6.3mm_D2.5mm_P2.54mm_Vertical, symbol Device:R
- added R10, R11, R8: 100K, Resistor_THT:R_Axial_DIN0207_L6.3mm_D2.5mm_P2.54mm_Vertical, symbol Device:R
- added R12, R13: 4,7K, Resistor_THT:R_Axial_DIN0207_L6.3mm_D2.5mm_P2.54mm_Vertical, symbol Device:R
- added R14, R15, R3, R5: 10K, Resistor_THT:R_Axial_DIN0207_L6.3mm_D2.5mm_P2.54mm_Vertical, symbol Device:R
- added R16, R17, R18: 220, Resistor_THT:R_Axial_DIN0207_L6.3mm_D2.5mm_P2.54mm_Vertical, symbol Device:R
- added R2: 720, Resistor_THT:R_Axial_DIN0207_L6.3mm_D2.5mm_P2.54mm_Vertical, symbol Device:R
- added R4, R6, R7: 470, Resistor_THT:R_Axial_DIN0207_L6.3mm_D2.5mm_P2.54mm_Vertical, symbol Device:R
- added R9: 390K, Resistor_THT:R_Axial_DIN0207_L6.3mm_D2.5mm_P2.54mm_Vertical, symbol Device:R
- added TP1, TP2, TP4, TP5: TestPoint, TestPoint:TestPoint_Pad_D1.0mm, symbol Connector:TestPoint
- added U1: ESP32_NODEMCU, JW_footprint_library:MODULE_ESP32_NODEMCU, symbol JW_library_sym:ESP32_NODEMCU
- added U2: LM317_TO-220, Package_TO_SOT_THT:TO-220-3_Vertical, symbol Regulator_Linear:LM317_TO-220
- added U3: LM358PE3, Package_DIP:DIP-8_W7.62mm_LongPads, symbol JW_library_sym:LM358PE3
- added U4, U5: TXS0108EPWR, TSSOP-20_4.4x5mm_P0.5mm, symbol JW_library_sym:TXS0108EPWR
- added Y1: 3.579546, Crystal:Crystal_HC49-4H_Vertical, symbol Device:Crystal
- J1: renamed from J?; footprint (none) -> Connector_BarrelJack:BarrelJack_Horizontal
Connections:
- net SDA: now also J3.1 (Pin_1), R13.2, U4.20 (B1)
- net at J1.1: now also C1.1, TP1.1, U2.3 (VI)
- net Earth: now reaches J1.2
- net Earth: now also C1.2, C2.2, C5.1, C7.2, C8.1, C9.1, D1.1 (K), D2.1 (K), D3.1 (K), D4.1 (K), D5.1 (K), H1.1, H2.1, H3.1, H4.1, IC1.5 (INH), IC1.9 (VSS), J2.2 (Pin_2), J2.3 (Pin_3), J2.4 (Pin_4), J2.5 (Pin_5), J3.7 (Pin_7), R2.2, R7.2, U1.J4_1 (GND_J4_1), U1.J4_7 (GND_J4_7), U1.J5_6 (GND_J5_6), U3.4 (GND), U4.11 (GND), U5.11 (GND)
- new net: C3.2, R3.2, R5.1, U3.2 (1IN-)
- new net: IC1.2 (IN-), R10.1, R8.1
- new net: IC1.3 (GS), R10.2
- new net: C10.1, R14.1, R15.2, U3.6 (2IN-)
- new net: IC1.11 (Q1), U5.1 (A1)
- new net: IC1.12 (Q2), U5.3 (A2)
- new net: IC1.13 (Q3), U5.4 (A3)
- new net: IC1.14 (Q4), U5.5 (A4)
- new net: C4.1, R8.2
- new net: D5.2 (A), R18.2
- new net: D1.2 (A), R4.2
- new net: C6.2, IC1.17 (ST/GT), R9.1
- new net: D3.2 (A), R16.1
- new net: D4.2 (A), R17.1
- new net: D2.2 (A), R11.2
- new net: IC1.15 (STD), R11.1
- new net: IC1.1 (IN+), IC1.4 (VREF)
- new net: IC1.16 (EST), R9.2
- new net: IC1.7 (OSC1), Y1.1
- new net: IC1.8 (OSC2), Y1.2
- new net: R1.1, R2.1, U2.1 (ADJ)
- new net 3V3: J2.1 (Pin_1), TP4.1, U1.J5_19 (3V3), U4.19 (VCCB), U5.19 (VCCB)
- new net 5V: C2.1, C6.1, C8.2, C9.2, IC1.10 (TOE), IC1.18 (VDD), J3.6 (Pin_6), R1.2, R12.1, R13.1, R4.1, R6.1, TP2.1, U1.J5_1 (5V), U2.2 (VO), U3.8 (VCC), U4.10 (OE), U4.2 (VCCA), U5.10 (OE), U5.2 (VCCA)
- new net Audio_ESP32: R14.2, U1.J5_11 (G25)
- new net Audio_ESP32-Amp: C10.2, R15.1, U3.7 (2OUT)
- new net Audio_SLIC: J3.5 (Pin_5), R3.1
- new net Audio_SLIC-Amp: C3.1, C4.2, R5.2, U3.1 (1OUT)
- new net Hook_Status_LED: R18.1, U1.J4_12 (G16)
- new net MCP_RESET: J3.4 (Pin_4), U4.16 (B4)
- new net MCP_RESET_3V: U1.J5_14 (G35), U4.5 (A4)
- new net MQTT_LED: R17.2, U1.J4_11 (G17)
- new net MT8870_PWDN: IC1.6 (PWDN), U5.6 (A5)
- new net MT8870_PWDN_3V: U1.J5_12 (G33), U5.15 (B5)
- new net Q1_3V: U1.J4_14 (G0), U5.20 (B1)
- new net Q2_3V: U1.J4_15 (G2), U5.18 (B2)
- new net Q3_3V: U1.J4_13 (G4), U5.17 (B3)
- new net Q4_3V: U1.J4_10 (G5), U5.16 (B4)
- new net SCL_3V: U1.J4_3 (G22), U4.3 (A2)
- new net SDA_3V: U1.J4_6 (G21), U4.1 (A1)
- new net SLC: J3.2 (Pin_2), R12.2, U4.18 (B2)
- new net SLIC_INT: J3.3 (Pin_3), U4.17 (B3)
- new net SLIC_INT_3V: U1.J5_15 (G34), U4.4 (A3)
- new net TCK: J2.7 (Pin_7), U1.J5_5 (G13)
- new net TDI: J2.9 (Pin_9), U1.J5_7 (G12)
- new net TDO: J2.8 (Pin_8), U1.J4_16 (G15)
- new net TMS: J2.6 (Pin_6), U1.J5_8 (G14)
- new net Vref: C5.2, C7.1, R6.2, R7.1, TP5.1, U3.3 (1IN+), U3.5 (2IN+)
- new net WiFi_LED: R16.2, U1.J4_9 (G18)
- no-connect marks 0 -> 31
Other:
- note added: "12V DC"
- note added: "Mounting holes"
- moved on the sheet: J1

Commit message: deleted:    KiCad/Exchange_ProofOfConcept/ESP-Unit/#auto_saved_files# 	modified:   KiCad/Exchange_ProofOfConcept/ESP-Unit/ESP-Unit.kicad_sch 	renamed:    KiCad/Exchange_ProofOfConcept/ESP-Unit/_autosave-ESP-Unit.kicad_sch -> KiCad/Exchange_ProofOfConcept/ESP-Unit/ESP-Unit.kicad_sch-bak 	new file:   KiCad/Exchange_ProofOfConcept/~Exchange_ProofOfConcept.kicad_pcb.lck 	new file:   KiCad/Exchange_ProofOfConcept/~Exchange_ProofOfConcept.kicad_sch.lck 	modified:   lib/MT8816/MT8816.cpp 	modified:   lib/MT8816/MT8816.h 	modified:   lib/RingHandler/RingHandler.cpp 	modified:   lib/RingHandler/RingHandler.h 	modified:   src/SHKhandler.h 	new file:   src/config.cpp 	modified:   src/config.h 	modified:   src/main.cpp
Parts:
- added C?: 2,2uF, Capacitor_THT:CP_Radial_D4.0mm_P2.00mm, symbol Device:C_Polarized_US
Connections:
- net 3V3: now also C?.1
- net at U1.J5_18 (EN): now also C?.2
Changed lines of the file:
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@@
 	(wire
 		(pts
+			(xy 30.48 77.47) (xy 30.48 81.28)
+		)
+		(stroke
+			(width 0)
+			(type default)
+		)
+	)
+	(wire
+		(pts
 			(xy 104.14 31.75) (xy 107.95 31.75)
 		)
@@
 	(wire
 		(pts
+			(xy 30.48 90.17) (xy 38.1 90.17)
+		)
+		(stroke
+			(width 0)
+			(type default)
+		)
+	)
+	(wire
+		(pts
 			(xy 113.03 110.49) (xy 113.03 105.41)
 		)
@@
 	(wire
 		(pts
+			(xy 30.48 88.9) (xy 30.48 90.17)
+		)
+		(stroke
+			(width 0)
+			(type default)
+		)
+	)
+	(wire
+		(pts
 			(xy 50.8 43.18) (xy 50.8 58.42)
 		)
@@
 		)
 	)
+	(label "3V3"
+		(at 30.48 77.47 0)
+		(fields_autoplaced yes)
+		(effects
+			(font
+				(size 1.27 1.27)
+			)
+			(justify left bottom)
+		)
+	)
 	(label "5V"
 		(at 182.88 35.56 180)
@@
 					(unit 1)
 				)
+			)
+		)
+	)
+	(symbol
+		(lib_id "Device:C_Polarized_US")
+		(at 30.48 85.09 0)
+		(unit 1)
+		(exclude_from_sim no)
+		(in_bom yes)
+		(on_board yes)
+		(dnp no)
+		(property "Reference" "C?"
+			(at 30.734 82.804 0)
+			(effects
+				(font
+					(size 1.27 1.27)
+				)
+				(justify left)
+			)
+		)
+		(property "Value" "2,2uF"
+			(at 30.988 87.884 0)
+			(effects
+				(font
+					(size 1.27 1.27)
+				)
+				(justify left)
+			)
+		)
+		(property "Footprint" "Capacitor_THT:CP_Radial_D4.0mm_P2.00mm"
+			(at 30.48 85.09 0)
+			(effects
+				(font
+					(size 1.27 1.27)
+				)
+				(hide yes)
+			)
+		)
+		(property "Datasheet" "~"
+			(at 30.48 85.09 0)
+			(effects
+				(font
+					(size 1.27 1.27)
+				)
+				(hide yes)
+			)
+		)
+		(property "Description" "Polarized capacitor, US symbol"
+			(at 30.48 85.09 0)
+			(effects
+				(font
+					(size 1.27 1.27)
+				)
+				(hide yes)
+			)
+		)
+		(pin "1"
+		)
+		(pin "2"
+		)
+		(instances
+			(project "ESP-Unit"
+				(path "/2411d7b8-ed2d-41a6-b5ea-3554d7cee414"
+					(reference "C?")
+					(unit 1)
+				)
