File: KiCad/Exchange_ProofOfConcept/ESP-Unit/ESP-Unit.kicad_sch (KiCad schematic)
At the start: 52 parts, among them IC1 MT8870DE, J1 Jack-DC, J2 Conn_02x05_Top_Bottom, J3 Conn_01x07, U1 ESP32_NODEMCU, U2 LM317_TO-220, U3 LM358PE3, U4 TXS0108EPWR, U5 TXS0108EPWR, Y1 3.579546

Commit message: Revert "RingHandlerDevelop"
Parts:
- removed C?: 2,2uF, Capacitor_THT:CP_Radial_D4.0mm_P2.00mm, symbol Device:C_Polarized_US
Connections:
- net Test_button: no longer names the net of U1.J4_8 (G19)
- no-connect marks 30 -> 31
Changed lines of the file:
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@@
 	)
 	(no_connect
+		(at 78.74 110.49)
+	)
+	(no_connect
 		(at 191.77 68.58)
 	)
@@
 	(wire
 		(pts
-			(xy 78.74 110.49) (xy 82.55 110.49)
-		)
-		(stroke
-			(width 0)
-			(type default)
-		)
-	)
-	(wire
-		(pts
 			(xy 162.56 100.33) (xy 160.02 100.33)
 		)
@@
 	(wire
 		(pts
-			(xy 30.48 77.47) (xy 30.48 81.28)
-		)
-		(stroke
-			(width 0)
-			(type default)
-		)
-	)
-	(wire
-		(pts
 			(xy 104.14 31.75) (xy 107.95 31.75)
 		)
@@
 	(wire
 		(pts
-			(xy 30.48 90.17) (xy 38.1 90.17)
-		)
-		(stroke
-			(width 0)
-			(type default)
-		)
-	)
-	(wire
-		(pts
 			(xy 113.03 110.49) (xy 113.03 105.41)
 		)
@@
 	(wire
 		(pts
-			(xy 30.48 88.9) (xy 30.48 90.17)
-		)
-		(stroke
-			(width 0)
-			(type default)
-		)
-	)
-	(wire
-		(pts
 			(xy 50.8 43.18) (xy 50.8 58.42)
 		)
@@
 		)
 	)
-	(label "3V3"
-		(at 30.48 77.47 0)
-		(fields_autoplaced yes)
-		(effects
-			(font
-				(size 1.27 1.27)
-			)
-			(justify left bottom)
-		)
-	)
 	(label "5V"
 		(at 182.88 35.56 180)
@@
 		)
 	)
-	(label "Test_button"
-		(at 82.55 110.49 0)
-		(fields_autoplaced yes)
-		(effects
-			(font
-				(size 1.27 1.27)
-			)
-			(justify left bottom)
-		)
-	)
 	(label "SLIC_INT"
 		(at 248.92 66.04 0)
@@
 					(unit 1)
 				)
-			)
-		)
-	)
-	(symbol
-		(lib_id "Device:C_Polarized_US")
-		(at 30.48 85.09 0)
-		(unit 1)
-		(exclude_from_sim no)
-		(in_bom yes)
-		(on_board yes)
-		(dnp no)
-		(property "Reference" "C?"
-			(at 30.734 82.804 0)
-			(effects
-				(font
-					(size 1.27 1.27)
-				)
-				(justify left)
-			)
-		)
-		(property "Value" "2,2uF"
-			(at 30.988 87.884 0)
-			(effects
-				(font
-					(size 1.27 1.27)
-				)
-				(justify left)
-			)
-		)
-		(property "Footprint" "Capacitor_THT:CP_Radial_D4.0mm_P2.00mm"
-			(at 30.48 85.09 0)
-			(effects
-				(font
-					(size 1.27 1.27)
-				)
-				(hide yes)
-			)
-		)
-		(property "Datasheet" "~"
-			(at 30.48 85.09 0)
-			(effects
-				(font
-					(size 1.27 1.27)
-				)
-				(hide yes)
-			)
-		)
-		(property "Description" "Polarized capacitor, US symbol"
-			(at 30.48 85.09 0)
-			(effects
-				(font
-					(size 1.27 1.27)
-				)
-				(hide yes)
-			)
-		)
-		(pin "1"
-		)
-		(pin "2"
-		)
-		(instances
-			(project "ESP-Unit"
-				(path "/2411d7b8-ed2d-41a6-b5ea-3554d7cee414"
-					(reference "C?")
-					(unit 1)
-				)
