File: KiCad/Exchange_ProofOfConcept/ESP-Unit/ESP-Unit.kicad_pcb (KiCad board)
At the start: 2 copper layers, 101.6 x 61.1 mm, 51 parts, among them IC1 MT8870DE, J1 Jack-DC, J2 Conn_02x05_Top_Bottom, J3 Conn_01x07, U1 ESP32_NODEMCU, U2 LM317_TO-220, U3 LM358PE3, U4 TXS0108EPWR, U5 TXS0108EPWR, Y1 3.579546

Commit message: deleted:    KiCad/Exchange_ProofOfConcept/ESP-Unit/ESP-Unit-backups/ESP-Unit-2024-10-22_204833.zip 	new file:   KiCad/Exchange_ProofOfConcept/ESP-Unit/ESP-Unit-backups/ESP-Unit-2025-01-21_222447.zip 	new file:   KiCad/Exchange_ProofOfConcept/ESP-Unit/ESP-Unit-backups/ESP-Unit-2025-01-23_205217.zip 	new file:   KiCad/Exchange_ProofOfConcept/ESP-Unit/ESP-Unit-backups/ESP-Unit-2025-01-23_211741.zip 	new file:   KiCad/Exchange_ProofOfConcept/ESP-Unit/ESP-Unit-backups/ESP-Unit-2025-01-26_102636.zip 	new file:   KiCad/Exchange_ProofOfConcept/ESP-Unit/ESP-Unit-backups/ESP-Unit-2025-01-30_220613.zip 	new file:   KiCad/Exchange_ProofOfConcept/ESP-Unit/ESP-Unit-backups/ESP-Unit-2025-01-30_221846.zip 	modified:   KiCad/Exchange_ProofOfConcept/ESP-Unit/ESP-Unit.kicad_pcb 	modified:   KiCad/Exchange_ProofOfConcept/ESP-Unit/ESP-Unit.kicad_pro 	modified:   KiCad/Exchange_ProofOfConcept/ESP-Unit/ESP-Unit.kicad_sch 	modified:   KiCad/Exchange_ProofOfConcept/ESP-Unit/fp-info-cache 	deleted:    KiCad/Exchange_ProofOfConcept/Exchange_ProofOfConcept-backups/Exchange_ProofOfConcept-2024-11-20_224852.zip 	deleted:    KiCad/Exchange_ProofOfConcept/Exchange_ProofOfConcept-backups/Exchange_ProofOfConcept-2024-11-20_230009.zip 	deleted:    KiCad/Exchange_ProofOfConcept/Exchange_ProofOfConcept-backups/Exchange_ProofOfConcept-2024-11-20_231023.zip 	deleted:    KiCad/Exchange_ProofOfConcept/Exchange_ProofOfConcept-backups/Exchange_ProofOfConcept-2024-11-20_231736.zip 	new file:   KiCad/Exchange_ProofOfConcept/Exchange_ProofOfConcept-backups/Exchange_ProofOfConcept-2025-01-21_210113.zip 	new file:   KiCad/Exchange_ProofOfConcept/Exchange_ProofOfConcept-backups/Exchange_ProofOfConcept-2025-01-21_210624.zip 	new file:   KiCad/Exchange_ProofOfConcept/Exchange_ProofOfConcept-backups/Exchange_ProofOfConcept-2025-01-21_214958.zip 	new file:   KiCad/Exchange_ProofOfConcept/Exchange_ProofOfConcept-backups/Exchange_ProofOfConcept-2025-01-21_222119.zip 	deleted:    KiCad/Exchange_ProofOfConcept/Exchange_Pr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
Parts:
- added C11: 0,1uF, Capacitor_THT:C_Disc_D5.0mm_W2.5mm_P2.50mm, F.Cu at (192.6, 34.3)
- C9: value 0,1uF -> 2,2uF; footprint Capacitor_THT:C_Disc_D5.0mm_W2.5mm_P2.50mm -> Capacitor_THT:CP_Radial_D4.0mm_P2.00mm
- U4, U5: value TXS0108EPWR -> BOB-12009; footprint Package_SO:TSSOP-20_4.4x5mm_P0.5mm -> JW_footprint_library:CONV_BOB-12009
- moved U5 43.6 mm to (235.7, 39.1)
- moved U4 25.4 mm to (210.6, 35.1)
Connections:
- C9 pad 1: Earth -> /3V3
- C9 pad 2: /5V -> unconnected-(C9-Pad2)
- IC1 pad 6: /MT8870_PWDN -> unconnected-(IC1-PWDN-Pad6)
- U1 pad J4_8: unconnected-(U1-G19-PadJ4_8) -> /Test_button
- U1 pad J5_12: /MT8870_PWDN_3V -> unconnected-(U1-G33-PadJ5_12)
- U1 pad J5_18: unconnected-(U1-EN-PadJ5_18) -> unconnected-(C9-Pad2)
Routing:
- net unconnected-(C9-Pad2): track 0.00 -> 3.50 mm
- net /5V: track 207.9 -> 204.4 mm
