File: KiCad/Exchange_ProofOfConcept/Exchange_ProofOfConcept.kicad_sch (KiCad schematic)
At the start: 29 parts, among them J1 Conn_02x03_Odd_Even, J2 Conn_02x03_Odd_Even, J7 Screw_Terminal_01x02, J9 Screw_Terminal_01x08, U1 MCP23017, U2 MCP23017, U3 MT8816

Commit message: modified:   .gitignore 	deleted:    KiCad/Exchange_ProofOfConcept/#auto_saved_files# 	deleted:    KiCad/Exchange_ProofOfConcept/Exchange_ProofOfConcept-backups/Exchange_ProofOfConcept-2024-10-11_163116.zip 	new file:   KiCad/Exchange_ProofOfConcept/Exchange_ProofOfConcept-backups/Exchange_ProofOfConcept-2024-11-27_224717.zip 	modified:   KiCad/Exchange_ProofOfConcept/Exchange_ProofOfConcept.kicad_sch 	deleted:    KiCad/Exchange_ProofOfConcept/_autosave-Exchange_ProofOfConcept.kicad_sch 	deleted:    KiCad/Exchange_ProofOfConcept/~Exchange_ProofOfConcept.kicad_pcb.lck 	deleted:    KiCad/Exchange_ProofOfConcept/~Exchange_ProofOfConcept.kicad_sch.lck 	new file:   lib/mqttHandler/secrets.h 	new file:   lib/mqttHandler/secrets.h.example
Parts:
- gave numbers to parts that had none: 1
Changed lines of the file:
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@@
 	)
 	(junction
-		(at 120.65 187.96)
-		(diameter 0)
-		(color 0 0 0 0)
-	)
-	(junction
 		(at 124.46 52.07)
 		(diameter 0)
@@
 		(color 0 0 0 0)
 	)
+	(junction
+		(at 120.65 187.96)
+		(diameter 0)
+		(color 0 0 0 0)
+	)
 	(no_connect
 		(at 270.51 71.12)
@@
 	(wire
 		(pts
-			(xy 120.65 187.96) (xy 125.73 187.96)
+			(xy 115.57 187.96) (xy 120.65 187.96)
 		)
 		(stroke
@@
 	(wire
 		(pts
-			(xy 115.57 187.96) (xy 120.65 187.96)
-		)
-		(stroke
-			(width 0)
-			(type default)
-		)
-	)
-	(wire
-		(pts
 			(xy 27.94 16.51) (xy 27.94 19.05)
 		)
@@
 	(wire
 		(pts
+			(xy 120.65 187.96) (xy 125.73 187.96)
+		)
+		(stroke
+			(width 0)
+			(type default)
+		)
+	)
+	(wire
+		(pts
 			(xy 223.52 147.32) (xy 231.14 147.32)
 		)
@@
 		(dnp no)
 		(fields_autoplaced yes)
-		(property "Reference" "J?"
+		(property "Reference" "J3"
 			(at 238.76 123.1899 0)
 			(effects
@@
 			(project ""
 				(path "/a3aa82f3-37b8-406c-999a-d11513c8e1fa"
-					(reference "J?")
+					(reference "J3")
 					(unit 1)
 				)
@@
 	)
 	(symbol
-		(lib_id "Mechanical:MountingHole_Pad")
-		(at 120.65 185.42 0)
+		(lib_id "power:GND")
+		(at 27.94 52.07 0)
 		(unit 1)
-		(exclude_from_sim yes)
-		(in_bom no)
+		(exclude_from_sim no)
+		(in_bom yes)
 		(on_board yes)
 		(dnp no)
 		(fields_autoplaced yes)
-		(property "Reference" "H2"
-			(at 123.19 182.8799 0)
+		(property "Reference" "#PWR01"
+			(at 27.94 58.42 0)
 			(effects
 				(font
 					(size 1.27 1.27)
 				)
-				(justify left)
 				(hide yes)
 			)
 		)
-		(property "Value" "MountingHole_Pad"
-			(at 123.19 185.4199 0)
+		(property "Value" "GND"
+			(at 27.94 57.15 0)
 			(effects
 				(font
 					(size 1.27 1.27)
 				)
-				(justify left)
-				(hide yes)
 			)
 		)
-		(property "Footprint" "MountingHole:MountingHole_3.2mm_M3_Pad_Via"
-			(at 120.65 185.42 0)
+		(property "Footprint" ""
+			(at 27.94 52.07 0)
 			(effects
 				(font
@@
 			)
 		)
-		(property "Datasheet" "~"
-			(at 120.65 185.42 0)
+		(property "Datasheet" ""
+			(at 27.94 52.07 0)
 			(effects
 				(font
@@
 			)
 		)
-		(property "Description" "Mounting Hole with connection"
-			(at 120.65 185.42 0)
+		(property "Description" "Power symbol creates a global label with name \"GND\" , ground"
+			(at 27.94 52.07 0)
 			(effects
 				(font
@@
 		)
 		(instances
-			(project "Exchange_ProofOfConcept"
+			(project ""
 				(path "/a3aa82f3-37b8-406c-999a-d11513c8e1fa"
-					(reference "H2")
+					(reference "#PWR01")
 					(unit 1)
 				)
@@
 	(symbol
 		(lib_id "power:GND")
-		(at 27.94 52.07 0)
+		(at 104.14 149.86 0)
 		(unit 1)
 		(exclude_from_sim no)
@@
 		(dnp no)
 		(fields_autoplaced yes)
-		(property "Reference" "#PWR01"
-			(at 27.94 58.42 0)
+		(property "Reference" "#PWR08"
+			(at 104.14 156.21 0)
 			(effects
 				(font
@@
 		)
 		(property "Value" "GND"
-			(at 27.94 57.15 0)
+			(at 104.14 154.94 0)
 			(effects
 				(font
@@
 		)
 		(property "Footprint" ""
-			(at 27.94 52.07 0)
+			(at 104.14 149.86 0)
 			(effects
 				(font
@@
 		)
 		(property "Datasheet" ""
-			(at 27.94 52.07 0)
+			(at 104.14 149.86 0)
 			(effects
 				(font
@@
 		)
 		(property "Description" "Power symbol creates a global label with name \"GND\" , ground"
-			(at 27.94 52.07 0)
+			(at 104.14 149.86 0)
 			(effects
 				(font
@@
 		)
 		(instances
-			(project ""
+			(project "Exchange_ProofOfConcept"
 				(path "/a3aa82f3-37b8-406c-999a-d11513c8e1fa"
-					(reference "#PWR01")
+					(reference "#PWR08")
 					(unit 1)
 				)
@@
 	)
 	(symbol
-		(lib_id "power:GND")
-		(at 104.14 149.86 0)
+		(lib_id "Mechanical:MountingHole_Pad")
+		(at 120.65 185.42 0)
 		(unit 1)
-		(exclude_from_sim no)
-		(in_bom yes)
+		(exclude_from_sim yes)
+		(in_bom no)
 		(on_board yes)
 		(dnp no)
 		(fields_autoplaced yes)
-		(property "Reference" "#PWR08"
-			(at 104.14 156.21 0)
+		(property "Reference" "H2"
+			(at 123.19 182.8799 0)
 			(effects
 				(font
 					(size 1.27 1.27)
 				)
+				(justify left)
 				(hide yes)
 			)
 		)
-		(property "Value" "GND"
-			(at 104.14 154.94 0)
+		(property "Value" "MountingHole_Pad"
+			(at 123.19 185.4199 0)
 			(effects
 				(font
 					(size 1.27 1.27)
 				)
+				(justify left)
+				(hide yes)
 			)
 		)
-		(property "Footprint" ""
-			(at 104.14 149.86 0)
+		(property "Footprint" "MountingHole:MountingHole_3.2mm_M3_Pad_Via"
+			(at 120.65 185.42 0)
 			(effects
 				(font
@@
 			)
 		)
-		(property "Datasheet" ""
-			(at 104.14 149.86 0)
+		(property "Datasheet" "~"
+			(at 120.65 185.42 0)
 			(effects
 				(font
@@
 			)
 		)
-		(property "Description" "Power symbol creates a global label with name \"GND\" , ground"
-			(at 104.14 149.86 0)
+		(property "Description" "Mounting Hole with connection"
+			(at 120.65 185.42 0)
 			(effects
 				(font
@@
 			(project "Exchange_ProofOfConcept"
 				(path "/a3aa82f3-37b8-406c-999a-d11513c8e1fa"
-					(reference "#PWR08")
+					(reference "H2")
 					(unit 1)
 				)

Commit message: Changes to be committed: 	new file:   KiCad/Exchange_ProofOfConcept/ESP-Unit/ESP-Unit-backups/ESP-Unit-2024-11-30_004013.zip 	new file:   KiCad/Exchange_ProofOfConcept/ESP-Unit/ESP-Unit-backups/ESP-Unit-2024-11-30_005151.zip 	new file:   KiCad/Exchange_ProofOfConcept/ESP-Unit/ESP-Unit-backups/ESP-Unit-2024-11-30_173159.zip 	new file:   KiCad/Exchange_ProofOfConcept/ESP-Unit/ESP-Unit-backups/ESP-Unit-2024-12-02_225320.zip 	new file:   KiCad/Exchange_ProofOfConcept/ESP-Unit/ESP-Unit-backups/ESP-Unit-2024-12-02_230401.zip 	new file:   KiCad/Exchange_ProofOfConcept/ESP-Unit/ESP-Unit-backups/ESP-Unit-2024-12-02_231401.zip 	new file:   KiCad/Exchange_ProofOfConcept/ESP-Unit/ESP-Unit-backups/ESP-Unit-2024-12-02_232414.zip 	new file:   KiCad/Exchange_ProofOfConcept/ESP-Unit/ESP-Unit-backups/ESP-Unit-2024-12-02_233354.zip 	new file:   KiCad/Exchange_ProofOfConcept/ESP-Unit/ESP-Unit-backups/ESP-Unit-2024-12-04_223019.zip 	new file:   KiCad/Exchange_ProofOfConcept/ESP-Unit/ESP-Unit-backups/ESP-Unit-2024-12-04_223655.zip 	new file:   KiCad/Exchange_ProofOfConcept/ESP-Unit/ESP-Unit-backups/ESP-Unit-2024-12-04_225021.zip 	new file:   KiCad/Exchange_ProofOfConcept/ESP-Unit/ESP-Unit-backups/ESP-Unit-2024-12-04_230524.zip 	new file:   KiCad/Exchange_ProofOfConcept/ESP-Unit/ESP-Unit-backups/ESP-Unit-2024-12-04_231506.zip 	new file:   KiCad/Exchange_ProofOfConcept/ESP-Unit/ESP-Unit-backups/ESP-Unit-2024-12-05_032122.zip 	new file:   KiCad/Exchange_ProofOfConcept/ESP-Unit/ESP-Unit-backups/ESP-Unit-2024-12-06_183750.zip 	new file:   KiCad/Exchange_ProofOfConcept/ESP-Unit/ESP-Unit-backups/ESP-Unit-2024-12-07_112304.zip 	new file:   KiCad/Exchange_ProofOfConcept/ESP-Unit/ESP-Unit-backups/ESP-Unit-2024-12-07_125326.zip 	modified:   KiCad/Exchange_ProofOfConcept/ESP-Unit/ESP-Unit.kicad_pcb 	modified:   KiCad/Exchange_ProofOfConcept/ESP-Unit/ESP-Unit.kicad_prl 	modified:   KiCad/Exchange_ProofOfConcept/ESP-Unit/ESP-Unit.kicad_pro 	modified:   KiCad/Exchange_ProofOfConcept/ESP-Unit/ESP-Unit.k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
Parts:
- removed J3: Conn_01x05, Connector_PinHeader_2.54mm:PinHeader_1x05_P2.54mm_Vertical, symbol Connector_Generic:Conn_01x05
- added J3: Conn_01x07, Connector_PinSocket_2.54mm:PinSocket_1x07_P2.54mm_Vertical, symbol Connector_Generic:Conn_01x07
Connections:
- net 5V: now also J3.6 (Pin_6)
- net Aout_x: now also J3.5 (Pin_5)
- net GND: now also J3.7 (Pin_7)
- net MCP_reset: now also J3.4 (Pin_4)
- net SCL: now also J3.2 (Pin_2)
- net SDA: now also J3.1 (Pin_1)
- net SLIC INT renamed SLIC_INT
- net SLIC_INT: now also J3.3 (Pin_3)
Other:
- moved on the sheet: J9

Commit message: deleted:    KiCad/Exchange_ProofOfConcept/#auto_saved_files# 	deleted:    KiCad/Exchange_ProofOfConcept/Exchange_ProofOfConcept-backups/Exchange_ProofOfConcept-2024-11-26_195718.zip 	new file:   KiCad/Exchange_ProofOfConcept/Exchange_ProofOfConcept-backups/Exchange_ProofOfConcept-2025-02-02_182812.zip 	modified:   KiCad/Exchange_ProofOfConcept/Exchange_ProofOfConcept.kicad_sch 	modified:   KiCad/Exchange_ProofOfConcept/SLIC 1.kicad_sch 	modified:   KiCad/Exchange_ProofOfConcept/SLIC 1_sch.kicad_sch 	modified:   KiCad/Exchange_ProofOfConcept/SLIC 3.kicad_sch 	modified:   KiCad/Exchange_ProofOfConcept/SLIC 4.kicad_sch 	deleted:    KiCad/Exchange_ProofOfConcept/_autosave-Exchange_ProofOfConcept.kicad_sch 	deleted:    KiCad/Exchange_ProofOfConcept/~Exchange_ProofOfConcept.kicad_pcb.lck 	deleted:    KiCad/Exchange_ProofOfConcept/~Exchange_ProofOfConcept.kicad_sch.lck 	modified:   docs/European harmonization of network generated tones.pdf 	modified:   include/config.h 	modified:   platformio.ini
Other:
- note added: "Detta behöver kopplas om så att Aout_0 hamnar på Y0 osv. Det blir onödigt krångligt i koden på detta sätt"
Changed lines of the file:
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@@
+		)
+	)
+	(polyline
+		(pts
+			(xy 273.05 73.66) (xy 273.05 92.71)
+		)
+		(stroke
+			(width 0)
+			(type default)
 		)
 	)
@@
 		)
 	)
+	(polyline
+		(pts
+			(xy 273.05 92.71) (xy 275.59 92.71)
+		)
+		(stroke
+			(width 0)
+			(type default)
+		)
+	)
 	(wire
 		(pts
@@
 			(width 0)
 			(type default)
+		)
+	)
+	(rectangle
+		(start 260.35 46.99)
+		(end 283.21 73.66)
+		(stroke
+			(width 0)
+			(type default)
+		)
+		(fill
+			(type none)
 		)
 	)
@@
 		)
 	)
+	(text "Detta behöver kopplas om så att Aout_0 hamnar på Y0 osv. \nDet blir onödigt krångligt i koden på detta sätt\n"
+		(exclude_from_sim no)
+		(at 276.352 95.504 0)
+		(effects
+			(font
+				(size 1.27 1.27)
+			)
+		)
+	)
 	(label "Ain_3"
 		(at 87.63 81.28 180)
-		(fields_autoplaced yes)
 		(effects
 			(font
@@
 	(label "Aout_x"
 		(at 275.59 63.5 0)
-		(fields_autoplaced yes)
 		(effects
 			(font
@@
 	(label "5V"
 		(at 17.78 143.51 0)
-		(fields_autoplaced yes)
 		(effects
 			(font
@@
 	(label "Aout_1"
 		(at 275.59 53.34 0)
-		(fields_autoplaced yes)
 		(effects
 			(font
@@
 	(label "Aout_1"
 		(at 45.72 34.29 0)
-		(fields_autoplaced yes)
 		(effects
 			(font
@@
 	(label "RING_2"
 		(at 45.72 69.85 0)
-		(fields_autoplaced yes)
 		(effects
 			(font
@@
 	(label "5V"
 		(at 171.45 21.59 0)
-		(fields_autoplaced yes)
 		(effects
 			(font
@@
 	(label "SCL"
 		(at 194.31 121.92 180)
-		(fields_autoplaced yes)
 		(effects
 			(font
@@
 	(label "5V"
 		(at 36.83 187.96 180)
-		(fields_autoplaced yes)
 		(effects
 			(font
@@
 	(label "Ain_2"
 		(at 228.6 88.9 270)
-		(fields_autoplaced yes)
 		(effects
 			(font
@@
 	(label "Aout_3"
 		(at 275.59 58.42 0)
-		(fields_autoplaced yes)
 		(effects
 			(font
@@
 	(label "RING_4"
 		(at 223.52 146.05 180)
-		(fields_autoplaced yes)
 		(effects
 			(font
@@
 	(label "Aout_3"
 		(at 87.63 78.74 180)
-		(fields_autoplaced yes)
 		(effects
 			(font
@@
 	(label "RING_3"
 		(at 87.63 72.39 180)
-		(fields_autoplaced yes)
 		(effects
 			(font
@@
 	(label "SDA"
 		(at 194.31 119.38 180)
-		(fields_autoplaced yes)
 		(effects
 			(font
@@
 	(label "TIP_4"
 		(at 223.52 143.51 180)
-		(fields_autoplaced yes)
 		(effects
 			(font
@@
 	(label "TIP_4"
 		(at 85.09 27.94 180)
-		(fields_autoplaced yes)
 		(effects
 			(font
@@
 	(label "Aout_2"
 		(at 275.59 55.88 0)
-		(fields_autoplaced yes)
 		(effects
 			(font
@@
 	(label "TIP_3"
 		(at 223.52 148.59 180)
-		(fields_autoplaced yes)
 		(effects
 			(font
@@
 	(label "RING_3"
 		(at 223.52 151.13 180)
-		(fields_autoplaced yes)
 		(effects
 			(font
@@
 	(label "Ain_1"
 		(at 226.06 88.9 270)
-		(fields_autoplaced yes)
 		(effects
 			(font
@@
 	(label "Aout_x"
 		(at 222.25 129.54 180)
-		(fields_autoplaced yes)
 		(effects
 			(font
@@
 	(label "5V"
 		(at 21.59 60.96 0)
-		(fields_autoplaced yes)
 		(effects
 			(font
@@
 	(label "Aout_4"
 		(at 85.09 34.29 180)
-		(fields_autoplaced yes)
 		(effects
 			(font
@@
 	(label "SLIC_INT"
 		(at 99.06 111.76 0)
-		(fields_autoplaced yes)
 		(effects
 			(font
@@
 	(label "Aout_4"
 		(at 275.59 60.96 0)
-		(fields_autoplaced yes)
 		(effects
 			(font
@@
 	(label "5V"
 		(at 107.95 60.96 0)
-		(fields_autoplaced yes)
 		(effects
 			(font
@@
 	(label "TIP_3"
 		(at 87.63 69.85 180)
-		(fields_autoplaced yes)
 		(effects
 			(font
@@
 	(label "SCL"
 		(at 139.7 78.74 180)
-		(fields_autoplaced yes)
 		(effects
 			(font
@@
 	(label "MCP_reset"
 		(at 222.25 127 180)
-		(fields_autoplaced yes)
 		(effects
 			(font
@@
 	(label "5V"
 		(at 222.25 132.08 180)
-		(fields_autoplaced yes)
 		(effects
 			(font
@@
 	(label "RING_2"
 		(at 223.52 156.21 180)
-		(fields_autoplaced yes)
 		(effects
 			(font
@@
 	(label "TIP_1"
 		(at 45.72 27.94 0)
-		(fields_autoplaced yes)
 		(effects
 			(font
@@
 	(label "TIP_1"
 		(at 223.52 158.75 180)
-		(fields_autoplaced yes)
 		(effects
 			(font
@@
 	(label "MCP_reset"
 		(at 135.89 30.48 90)
-		(fields_autoplaced yes)
 		(effects
 			(font
@@
 	(label "Aout_2"
 		(at 45.72 78.74 0)
-		(fields_autoplaced yes)
 		(effects
 			(font
@@
 	(label "5V"
 		(at 127 30.48 180)
-		(fields_autoplaced yes)
 		(effects
 			(font
@@
 	(label "RING_1"
 		(at 223.52 161.29 180)
-		(fields_autoplaced yes)
 		(effects
 			(font
@@
 	(label "Ain_4"
 		(at 85.09 36.83 180)
-		(fields_autoplaced yes)
 		(effects
 			(font
@@
 	(label "TIP_2"
 		(at 45.72 72.39 0)
-		(fields_autoplaced yes)
 		(effects
 			(font
@@
 	(label "MCP_reset"
 		(at 36.83 179.07 180)
-		(fields_autoplaced yes)
 		(effects
 			(font
@@
 	(label "Ain_4"
 		(at 233.68 88.9 270)
-		(fields_autoplaced yes)
 		(effects
 			(font
@@
 	(label "Ain_2"
 		(at 45.72 81.28 0)
-		(fields_autoplaced yes)
 		(effects
 			(font
@@
 	(label "Ain_1"
 		(at 45.72 36.83 0)
-		(fields_autoplaced yes)
 		(effects
 			(font
@@
 	(label "5V"
 		(at 27.94 16.51 0)
-		(fields_autoplaced yes)
 		(effects
 			(font
@@
 	(label "Ain_3"
 		(at 231.14 88.9 270)
-		(fields_autoplaced yes)
 		(effects
 			(font
@@
 	(label "5V"
 		(at 165.1 106.68 180)
-		(fields_autoplaced yes)
 		(effects
 			(font
@@
 	(label "RING_1"
 		(at 45.72 25.4 0)
-		(fields_autoplaced yes)
 		(effects
 			(font
@@
 	(label "5V"
 		(at 102.87 16.51 0)
-		(fields_autoplaced yes)
 		(effects
 			(font
@@
 	(label "5V"
 		(at 205.74 153.67 180)
-		(fields_autoplaced yes)
 		(effects
 			(font
@@
 	(label "SDA"
 		(at 82.55 171.45 270)
-		(fields_autoplaced yes)
 		(effects
 			(font
@@
 	(label "RING_4"
 		(at 85.09 25.4 180)
-		(fields_autoplaced yes)
 		(effects
 			(font
@@
 	(label "SDA"
 		(at 139.7 76.2 180)
-		(fields_autoplaced yes)
 		(effects
 			(font
@@
 	(label "SLIC_INT"
 		(at 222.25 124.46 180)
-		(fields_autoplaced yes)
 		(effects
 			(font
@@
 	(label "SCL"
 		(at 85.09 171.45 270)
-		(fields_autoplaced yes)
 		(effects
 			(font
@@
 	(label "5V"
 		(at 245.11 26.67 0)
-		(fields_autoplaced yes)
 		(effects
 			(font
@@
 	(label "TIP_2"
 		(at 223.52 153.67 180)
-		(fields_autoplaced yes)
 		(effects
 			(font
@@
 	(label "GND"
 		(at 165.1 111.76 180)
-		(fields_autoplaced yes)
-		(effects
-			(font
+		(effects
+			(font

Commit message: Revert "Number dailing"
Other:
- note removed: "Detta behöver kopplas om så att Aout_0 hamnar på Y0 osv. Det blir onödigt krångligt i koden på detta sätt"
Changed lines of the file:
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@@
-		)
-	)
-	(polyline
-		(pts
-			(xy 273.05 73.66) (xy 273.05 92.71)
-		)
-		(stroke
-			(width 0)
-			(type default)
 		)
 	)
@@
 		)
 	)
-	(polyline
-		(pts
-			(xy 273.05 92.71) (xy 275.59 92.71)
-		)
-		(stroke
-			(width 0)
-			(type default)
-		)
-	)
 	(wire
 		(pts
@@
 			(width 0)
 			(type default)
-		)
-	)
-	(rectangle
-		(start 260.35 46.99)
-		(end 283.21 73.66)
-		(stroke
-			(width 0)
-			(type default)
-		)
-		(fill
-			(type none)
 		)
 	)
@@
 		)
 	)
-	(text "Detta behöver kopplas om så att Aout_0 hamnar på Y0 osv. \nDet blir onödigt krångligt i koden på detta sätt\n"
-		(exclude_from_sim no)
-		(at 276.352 95.504 0)
-		(effects
-			(font
-				(size 1.27 1.27)
-			)
-		)
-	)
 	(label "Ain_3"
 		(at 87.63 81.28 180)
+		(fields_autoplaced yes)
 		(effects
 			(font
@@
 	(label "Aout_x"
 		(at 275.59 63.5 0)
+		(fields_autoplaced yes)
 		(effects
 			(font
@@
 	(label "5V"
 		(at 17.78 143.51 0)
+		(fields_autoplaced yes)
 		(effects
 			(font
@@
 	(label "Aout_1"
 		(at 275.59 53.34 0)
+		(fields_autoplaced yes)
 		(effects
 			(font
@@
 	(label "Aout_1"
 		(at 45.72 34.29 0)
+		(fields_autoplaced yes)
 		(effects
 			(font
@@
 	(label "RING_2"
 		(at 45.72 69.85 0)
+		(fields_autoplaced yes)
 		(effects
 			(font
@@
 	(label "5V"
 		(at 171.45 21.59 0)
+		(fields_autoplaced yes)
 		(effects
 			(font
@@
 	(label "SCL"
 		(at 194.31 121.92 180)
+		(fields_autoplaced yes)
 		(effects
 			(font
@@
 	(label "5V"
 		(at 36.83 187.96 180)
+		(fields_autoplaced yes)
 		(effects
 			(font
@@
 	(label "Ain_2"
 		(at 228.6 88.9 270)
+		(fields_autoplaced yes)
 		(effects
 			(font
@@
 	(label "Aout_3"
 		(at 275.59 58.42 0)
+		(fields_autoplaced yes)
 		(effects
 			(font
@@
 	(label "RING_4"
 		(at 223.52 146.05 180)
+		(fields_autoplaced yes)
 		(effects
 			(font
@@
 	(label "Aout_3"
 		(at 87.63 78.74 180)
+		(fields_autoplaced yes)
 		(effects
 			(font
@@
 	(label "RING_3"
 		(at 87.63 72.39 180)
+		(fields_autoplaced yes)
 		(effects
 			(font
@@
 	(label "SDA"
 		(at 194.31 119.38 180)
+		(fields_autoplaced yes)
 		(effects
 			(font
@@
 	(label "TIP_4"
 		(at 223.52 143.51 180)
+		(fields_autoplaced yes)
 		(effects
 			(font
@@
 	(label "TIP_4"
 		(at 85.09 27.94 180)
+		(fields_autoplaced yes)
 		(effects
 			(font
@@
 	(label "Aout_2"
 		(at 275.59 55.88 0)
+		(fields_autoplaced yes)
 		(effects
 			(font
@@
 	(label "TIP_3"
 		(at 223.52 148.59 180)
+		(fields_autoplaced yes)
 		(effects
 			(font
@@
 	(label "RING_3"
 		(at 223.52 151.13 180)
+		(fields_autoplaced yes)
 		(effects
 			(font
@@
 	(label "Ain_1"
 		(at 226.06 88.9 270)
+		(fields_autoplaced yes)
 		(effects
 			(font
@@
 	(label "Aout_x"
 		(at 222.25 129.54 180)
+		(fields_autoplaced yes)
 		(effects
 			(font
@@
 	(label "5V"
 		(at 21.59 60.96 0)
+		(fields_autoplaced yes)
 		(effects
 			(font
@@
 	(label "Aout_4"
 		(at 85.09 34.29 180)
+		(fields_autoplaced yes)
 		(effects
 			(font
@@
 	(label "SLIC_INT"
 		(at 99.06 111.76 0)
+		(fields_autoplaced yes)
 		(effects
 			(font
@@
 	(label "Aout_4"
 		(at 275.59 60.96 0)
+		(fields_autoplaced yes)
 		(effects
 			(font
@@
 	(label "5V"
 		(at 107.95 60.96 0)
+		(fields_autoplaced yes)
 		(effects
 			(font
@@
 	(label "TIP_3"
 		(at 87.63 69.85 180)
+		(fields_autoplaced yes)
 		(effects
 			(font
@@
 	(label "SCL"
 		(at 139.7 78.74 180)
+		(fields_autoplaced yes)
 		(effects
 			(font
@@
 	(label "MCP_reset"
 		(at 222.25 127 180)
+		(fields_autoplaced yes)
 		(effects
 			(font
@@
 	(label "5V"
 		(at 222.25 132.08 180)
+		(fields_autoplaced yes)
 		(effects
 			(font
@@
 	(label "RING_2"
 		(at 223.52 156.21 180)
+		(fields_autoplaced yes)
 		(effects
 			(font
@@
 	(label "TIP_1"
 		(at 45.72 27.94 0)
+		(fields_autoplaced yes)
 		(effects
 			(font
@@
 	(label "TIP_1"
 		(at 223.52 158.75 180)
+		(fields_autoplaced yes)
 		(effects
 			(font
@@
 	(label "MCP_reset"
 		(at 135.89 30.48 90)
+		(fields_autoplaced yes)
 		(effects
 			(font
@@
 	(label "Aout_2"
 		(at 45.72 78.74 0)
+		(fields_autoplaced yes)
 		(effects
 			(font
@@
 	(label "5V"
 		(at 127 30.48 180)
+		(fields_autoplaced yes)
 		(effects
 			(font
@@
 	(label "RING_1"
 		(at 223.52 161.29 180)
+		(fields_autoplaced yes)
 		(effects
 			(font
@@
 	(label "Ain_4"
 		(at 85.09 36.83 180)
+		(fields_autoplaced yes)
 		(effects
 			(font
@@
 	(label "TIP_2"
 		(at 45.72 72.39 0)
+		(fields_autoplaced yes)
 		(effects
 			(font
@@
 	(label "MCP_reset"
 		(at 36.83 179.07 180)
+		(fields_autoplaced yes)
 		(effects
 			(font
@@
 	(label "Ain_4"
 		(at 233.68 88.9 270)
+		(fields_autoplaced yes)
 		(effects
 			(font
@@
 	(label "Ain_2"
 		(at 45.72 81.28 0)
+		(fields_autoplaced yes)
 		(effects
 			(font
@@
 	(label "Ain_1"
 		(at 45.72 36.83 0)
+		(fields_autoplaced yes)
 		(effects
 			(font
@@
 	(label "5V"
 		(at 27.94 16.51 0)
+		(fields_autoplaced yes)
 		(effects
 			(font
@@
 	(label "Ain_3"
 		(at 231.14 88.9 270)
+		(fields_autoplaced yes)
 		(effects
 			(font
@@
 	(label "5V"
 		(at 165.1 106.68 180)
+		(fields_autoplaced yes)
 		(effects
 			(font
@@
 	(label "RING_1"
 		(at 45.72 25.4 0)
+		(fields_autoplaced yes)
 		(effects
 			(font
@@
 	(label "5V"
 		(at 102.87 16.51 0)
+		(fields_autoplaced yes)
 		(effects
 			(font
@@
 	(label "5V"
 		(at 205.74 153.67 180)
+		(fields_autoplaced yes)
 		(effects
 			(font
@@
 	(label "SDA"
 		(at 82.55 171.45 270)
+		(fields_autoplaced yes)
 		(effects
 			(font
@@
 	(label "RING_4"
 		(at 85.09 25.4 180)
+		(fields_autoplaced yes)
 		(effects
 			(font
@@
 	(label "SDA"
 		(at 139.7 76.2 180)
+		(fields_autoplaced yes)
 		(effects
 			(font
@@
 	(label "SLIC_INT"
 		(at 222.25 124.46 180)
+		(fields_autoplaced yes)
 		(effects
 			(font
@@
 	(label "SCL"
 		(at 85.09 171.45 270)
+		(fields_autoplaced yes)
 		(effects
 			(font
@@
 	(label "5V"
 		(at 245.11 26.67 0)
+		(fields_autoplaced yes)
 		(effects
 			(font
@@
 	(label "TIP_2"
 		(at 223.52 153.67 180)
+		(fields_autoplaced yes)
 		(effects
 			(font
@@
 	(label "GND"
 		(at 165.1 111.76 180)
-		(effects
-			(font
+		(fields_autoplaced yes)
+		(effects
+			(font
