File: KiCad/Exchange_ProofOfConcept/_autosave-Exchange_ProofOfConcept.kicad_sch (KiCad schematic)
At the start: 29 parts, among them J1 Conn_02x03_Odd_Even, J2 Conn_02x03_Odd_Even, J3 Conn_01x07, J7 Screw_Terminal_01x02, J9 Screw_Terminal_01x08, U1 MCP23017, U2 MCP23017, U3 MT8816

Commit message: Revert "Number dailing"
Other:
- note removed: "Aout_X borde döpas om och läggas bland en utav X-ingångarna"
- note removed: "Linjerna behöver byta namn och förskjutas 1 steg så att line 1 istället blir line 0 osv. Detta linjerar bättre med koden"
Changed lines of the file:
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@@
-		)
-	)
-	(text "Linjerna behöver byta namn och förskjutas 1 steg så att line 1 istället blir line 0 osv. \nDetta linjerar bättre med koden"
-		(exclude_from_sim no)
-		(at 64.77 5.588 0)
-		(effects
-			(font
-				(size 1.27 1.27)
-			)
 		)
 	)
@@
 		(effects
 			(font
-				(size 1.27 1.27)
-			)
-		)
-	)
-	(text "Aout_X borde döpas om och läggas bland en utav X-ingångarna"
-		(exclude_from_sim no)
-		(at 320.548 62.738 0)
-		(effects
-			(font
